File: eagle/altimeter.brd (EAGLE design)
At the start: 99.1 x 74.9 mm, 34 parts, among them U1 328P

Commit message: Created project structure and updated eagle files
Routing:
- net N$8: track 21.2 -> 29.2 mm
- net N$9: track 21.2 -> 27.9 mm
- net DROUGEREAD: track 26.0 -> 27.6 mm
- net GND: track 316.3 -> 315.7 mm
- net DROUGEDEPLOY: vias 0 -> 1
