File: eagle/altimeter.sch (EAGLE design)
At the start: 34 parts, among them U1 328P

Commit message: Created project structure and updated eagle files
Other:
- moved on the sheet: BMP280, DROUGE, DROUGETERMINAL, ERROR, FRAMTERM, LOOP, LOOPSTOP, LS1, MAIN, MAINTERMINAL, POWER, Q1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
